File: LM5116 Kicad File/LM5116.kicad_pcb (KiCad board)
At the start: 4 copper layers, 58.5 x 83.3 mm, 84 parts, among them J1 XT60-M, J10 PH1-01-UA, J11 PH1-01-UA, J12 PH1-01-UA, J13 PH1-01-UA, J14 61300311121, J15 61300311121, J16 61300311121, J17 61300311121, J18 61300311121, J19 61300311121, J2 PH1-01-UA, J20 61300311121, J21 61300311121, J22 61300311121, J23 61300311121, J24 61300311121, J25 61300311121, J3 PH1-01-UA, J4 PH1-01-UA, J5 PH1-01-UA, J6 PH1-01-UA, J7 PH1-01-UA, J8 PH1-01-UA, J9 PH1-01-UA, Q1 CSD17304Q3, Q2 CSD17304Q3, Q3 CSD17304Q3, Q4 CSD17304Q3, Q5 2N7002, Q6 IQDH29NE2LM5CG, U1 LM25116MHX/NOPB, U2 TLV1701AIDBVR, U3 TL431DBZ

Commit message: New Kicad File Final
Parts:
- C4: value 100u -> 680u; footprint Capacitor_SMD:CP_Elec_6.3x5.8 -> Capacitor_SMD:CP_Elec_10x10.5
- moved J14 50.8 mm to (172.7, 119.6), turned to 90 degrees
- moved J2 50.7 mm to (172.7, 125.7), turned to 0 degrees
- moved J25 48.3 mm to (123.2, 119.4), turned to 90 degrees
- moved J8 48.3 mm to (123.2, 125.7), turned to 0 degrees
- moved J15 41.9 mm to (168.3, 119.6), turned to 90 degrees
- moved J3 41.9 mm to (168.3, 125.7), turned to 0 degrees
- moved J24 39.4 mm to (127.6, 119.6), turned to 90 degrees
- moved J9 39.4 mm to (127.6, 125.7), turned to 0 degrees
- moved J16 33.0 mm to (163.8, 119.6), turned to 90 degrees
- moved J4 33.0 mm to (163.8, 125.7), turned to 0 degrees
- moved J10 29.2 mm to (132.7, 125.7), turned to 0 degrees
- moved J23 29.2 mm to (132.7, 119.6), turned to 90 degrees
- moved J17 24.1 mm to (159.4, 119.6), turned to 90 degrees
- moved J5 24.1 mm to (159.4, 125.7), turned to 0 degrees
- moved J11 20.3 mm to (137.2, 125.7), turned to 0 degrees
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Connections:
- C1 pad 2: GNDPWR -> GND
- C10 pad 2: GNDPWR -> GND
- C2 pad 2: GNDPWR -> GND
- C21 pad 2: GNDPWR -> GND
- C3 pad 2: GNDPWR -> GND
- C6 pad 2: GNDPWR -> GND
- C7 pad 2: GNDPWR -> GND
- C8 pad 2: GNDPWR -> GND
- J14 pad 1: /VOUT -> /1
- J14 pad 2: /1 -> /VOUT
- J15 pad 1: /VOUT -> /2
- J15 pad 2: /2 -> /VOUT
- J16 pad 1: /VOUT -> /3
- J16 pad 2: /3 -> /VOUT
- J17 pad 1: /VOUT -> /4
- J17 pad 2: /4 -> /VOUT
- J18 pad 1: /VOUT -> /5
- J18 pad 2: /5 -> /VOUT
- J19 pad 1: /VOUT -> /6
- J19 pad 2: /6 -> /VOUT
- J20 pad 1: /VOUT -> /12
- J20 pad 2: /12 -> /VOUT
- J21 pad 1: /VOUT -> /11
- J21 pad 2: /11 -> /VOUT
- J22 pad 1: /VOUT -> /10
- J22 pad 2: /10 -> /VOUT
- J23 pad 1: /VOUT -> /9
- J23 pad 2: /9 -> /VOUT
- J24 pad 1: /VOUT -> /8
- J24 pad 2: /8 -> /VOUT
- J25 pad 1: /VOUT -> /7
- J25 pad 2: /7 -> /VOUT
- Q5 pad 2: GNDPWR -> GND
- R1 pad 2: GNDPWR -> GND
- R20 pad 2: GNDPWR -> GND
- R5 pad 2: GNDPWR -> GND
- R9 pad 2: GNDPWR -> GND
- U1 pad 6: GNDPWR -> GND
- U3 pad 3: GNDPWR -> GND
Routing:
- net /VOUT: track 127.6 -> 212.2 mm, vias 7 -> 8
- net GNDPWR: track 112.1 -> 80.4 mm, vias 89 -> 72
- net GND: track 0.00 -> 20.3 mm, vias 0 -> 15
- net /8: track 7.91 -> 3.58 mm
- net /9: track 7.70 -> 3.58 mm
- net /6: track 7.70 -> 3.58 mm
- net /4: track 7.70 -> 3.58 mm
- net /2: track 7.70 -> 3.58 mm
- net /11: track 7.70 -> 3.58 mm
- net /1: track 7.60 -> 3.59 mm
- net /5: track 7.59 -> 3.58 mm
- net /3: track 7.59 -> 3.58 mm
- net /10: track 7.59 -> 3.58 mm
- net /7: track 7.82 -> 4.04 mm
- net /12: track 7.14 -> 3.58 mm
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Other:
- board text added: "EX"
- board text added: "OFF"
- board text added: "ON"
- board text added: "VIN"
- board text removed: "+6.8V"
