File: LM5116 Kicad File/LM5116.kicad_pcb (KiCad board)
At the start: 4 copper layers, 58.5 x 83.3 mm, 84 parts, among them J1 XT60-M, J10 PH1-01-UA, J11 PH1-01-UA, J12 PH1-01-UA, J13 PH1-01-UA, J14 61300311121, J15 61300311121, J16 61300311121, J17 61300311121, J18 61300311121, J19 61300311121, J2 PH1-01-UA, J20 61300311121, J21 61300311121, J22 61300311121, J23 61300311121, J24 61300311121, J25 61300311121, J3 PH1-01-UA, J4 PH1-01-UA, J5 PH1-01-UA, J6 PH1-01-UA, J7 PH1-01-UA, J8 PH1-01-UA, J9 PH1-01-UA, Q1 CSD17304Q3, Q2 CSD17304Q3, Q3 CSD17304Q3, Q4 CSD17304Q3, Q5 2N7002, Q6 IQDH29NE2LM5CG, U1 LM25116MHX/NOPB, U2 TLV1701AIDBVR, U3 TL431DBZ

Commit message: Update Footprint
Parts:
- moved Q1 7.56 mm to (154.5, 75.1)
- moved Q2 7.56 mm to (149.5, 75.1)
- moved C12 7.56 mm to (155.4, 112.6)
- moved C13 7.56 mm to (143.4, 113.0)
- moved C17 7.56 mm to (157.4, 120.5)
- moved C20 7.56 mm to (139.6, 89.8)
- moved C7 7.56 mm to (139.6, 79.6)
- moved C9 7.56 mm to (151.0, 79.6)
- moved D3 7.56 mm to (152.9, 78.9)
- moved J12 7.56 mm to (145.3, 132.3)
- moved J17 7.56 mm to (163.1, 126.2)
- moved J21 7.56 mm to (145.3, 126.2)
- moved J5 7.56 mm to (163.1, 132.3)
- moved R13 7.56 mm to (149.1, 79.6)
- moved R17 7.56 mm to (147.2, 89.7)
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Routing:
- net GNDPWR: track 80.4 -> 65.4 mm
- added copper zone on F.Cu, net GNDPWR
Other:
- board outline removed

Commit message: Update Kicad File
Parts:
- C2: value 220p -> 180p; footprint Capacitor_SMD:C_0603_1608Metric_Pad1.08x0.95mm_HandSolder -> Capacitor_SMD:C_0402_1005Metric_Pad0.74x0.62mm_HandSolder
- C3: value 100p -> 33n; footprint Capacitor_SMD:C_0201_0603Metric_Pad0.64x0.40mm_HandSolder -> Capacitor_SMD:C_0805_2012Metric_Pad1.18x1.45mm_HandSolder
- R2: value 10k -> 22.6k
- R3: value 1.5k -> 2.49k; footprint Resistor_SMD:R_0402_1005Metric_Pad0.72x0.64mm_HandSolder -> Resistor_SMD:R_0603_1608Metric_Pad0.98x0.95mm_HandSolder
- R5: value 10.2k -> 5.3k; footprint Resistor_SMD:R_0805_2012Metric_Pad1.20x1.40mm_HandSolder -> Resistor_SMD:R_0603_1608Metric_Pad0.98x0.95mm_HandSolder
- moved R3 7.89 mm to (133.3, 73.7)
- moved Q1 7.56 mm to (150.8, 68.5)
- moved Q2 7.56 mm to (145.8, 68.5)
- moved C12 7.56 mm to (151.8, 106.0)
- moved C13 7.56 mm to (139.7, 106.4)
- moved C17 7.56 mm to (153.7, 113.9)
- moved C7 7.56 mm to (135.9, 73.0)
- moved C9 7.56 mm to (147.4, 73.0)
- moved D3 7.56 mm to (149.3, 72.3)
- moved J12 7.56 mm to (141.6, 125.7)
- moved J17 7.56 mm to (159.4, 119.6)
- moved J21 7.56 mm to (141.6, 119.6)
- moved J5 7.56 mm to (159.4, 125.7)
- moved R13 7.56 mm to (145.5, 73.0)
- moved R17 7.56 mm to (143.5, 83.1)
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Routing:
- net GNDPWR: track 65.4 -> 80.4 mm
- net /RT_SYNC: track 6.44 -> 7.53 mm
- net GND: track 20.3 -> 21.1 mm
- net Net-(U1-SS): track 3.31 -> 2.67 mm
- net Net-(U1-RAMP): track 5.16 -> 5.61 mm, vias 2 -> 0
- net /SW: vias 39 -> 41
- removed copper zone on F.Cu, net GNDPWR
Other:
- board outline added: 58.5 x 83.3 mm
