File: Ai Sipder Bot Power System/LM5116 Kicad File/LM5116.kicad_pcb (KiCad board)
At the start: 4 copper layers, 60.2 x 83.5 mm, 89 parts, among them J1 XT60-M, J10 PH1-01-UA, J11 PH1-01-UA, J12 PH1-01-UA, J13 PH1-01-UA, J14 61300311121, J15 61300311121, J16 61300311121, J17 61300311121, J18 61300311121, J19 61300311121, J2 PH1-01-UA, J20 61300311121, J21 61300311121, J22 61300311121, J23 61300311121, J24 61300311121, J25 61300311121, J26 691137710002, J3 PH1-01-UA, J4 PH1-01-UA, J5 PH1-01-UA, J6 PH1-01-UA, J7 PH1-01-UA, J8 PH1-01-UA, J9 PH1-01-UA, Q1 CSD17304Q3, Q2 CSD17304Q3, Q3 CSD17304Q3, Q4 CSD17304Q3, Q5 2N7002, Q6 IQDH29NE2LM5CG, U1 LM25116MHX/NOPB, U2 TLV1701AIDBVR, U3 TL431DBZ

Commit message: Update Gerber File
Parts:
- moved C5 13.1 mm to (151.5, 74.3)
- moved F1 2.07 mm to (131.4, 66.2)
- moved Q3 1.13 mm to (148.0, 90.1), turned to 180 degrees
- moved C1 0.88 mm to (148.4, 83.4)
- moved Q2 0.64 mm to (142.5, 75.0), turned to -90 degrees
- moved R25 0.17 mm to (143.4, 78.3), turned to -90 degrees
- turned Q1 to -90 degrees
- turned Q4 to -90 degrees
Connections:
- C1 pad 2: GND -> GNDPWR
- C10 pad 2: GND -> GNDPWR
Routing:
- net GNDPWR: track 55.9 -> 70.3 mm, vias 77 -> 96
- net /CS: track 11.1 -> 19.6 mm
- net Net-(Q3-Gate): track 3.46 -> 11.9 mm, vias 0 -> 2
- net /SW: track 12.8 -> 8.49 mm, vias 25 -> 24
- net Net-(Q4-Gate): track 6.36 -> 10.6 mm, vias 0 -> 2
- net Net-(Q1-Gate): track 3.70 -> 6.34 mm
- net Net-(Q2-Gate): track 3.57 -> 5.96 mm
- net GND: track 12.0 -> 11.0 mm, vias 34 -> 32
- net /VOUT: track 212.7 -> 213.4 mm
Other:
- board size 60.2 x 83.5 mm -> 60.3 x 83.5 mm

Commit message: Add Gerber File
Parts:
- moved C5 0.85 mm to (151.5, 75.1)
Routing:
- net GNDPWR: vias 96 -> 77
- net /VOUT: vias 7 -> 33
- net /SW: vias 24 -> 20
- net /SOURCE: vias 3 -> 23
- added copper zone on F.Cu, net /SOURCE
- added copper zone on F.Cu, net /VOUT
Other:
- board size 60.3 x 83.5 mm -> 72.4 x 83.5 mm

Commit message: Update gerber
Routing:
- net /VOUT: vias 33 -> 18
- net /SOURCE: vias 23 -> 15
Changed lines of the file:
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@@
 	)
 	(via
-		(at 140.9954 100.206315)
+		(at 138.791631 100.505291)
 		(size 0.6)
 		(drill 0.3)
@@
 	)
 	(via
-		(at 139.69492 96.529)
+		(at 138.791631 96.441291)
 		(size 0.6)
 		(drill 0.3)
@@
 	)
 	(via
-		(at 183.241631 125.901145)
-		(size 0.6)
-		(drill 0.3)
-		(layers "F.Cu" "B.Cu")
-		(free yes)
-		(net "/VOUT")
-	)
-	(via
-		(at 115.779231 116.784618)
-		(size 0.6)
-		(drill 0.3)
-		(layers "F.Cu" "B.Cu")
-		(free yes)
-		(net "/VOUT")
-	)
-	(via
-		(at 115.779231 113.64331)
-		(size 0.6)
-		(drill 0.3)
-		(layers "F.Cu" "B.Cu")
-		(free yes)
-		(net "/VOUT")
-	)
-	(via
-		(at 183.241631 122.747399)
-		(size 0.6)
-		(drill 0.3)
-		(layers "F.Cu" "B.Cu")
-		(free yes)
-		(net "/VOUT")
-	)
-	(via
 		(at 183.241631 121.176745)
 		(size 0.6)
@@
 	)
 	(via
-		(at 117.557231 116.784618)
-		(size 0.6)
-		(drill 0.3)
-		(layers "F.Cu" "B.Cu")
-		(free yes)
-		(net "/VOUT")
-	)
-	(via
-		(at 183.241631 127.471799)
-		(size 0.6)
-		(drill 0.3)
-		(layers "F.Cu" "B.Cu")
-		(free yes)
-		(net "/VOUT")
-	)
-	(via
-		(at 180.100323 129.054891)
-		(size 0.6)
-		(drill 0.3)
-		(layers "F.Cu" "B.Cu")
-		(free yes)
-		(net "/VOUT")
-	)
-	(via
 		(at 129.3622 91.068)
 		(size 0.6)
@@
 	)
 	(via
-		(at 117.557231 113.643311)
-		(size 0.6)
-		(drill 0.3)
-		(layers "F.Cu" "B.Cu")
-		(free yes)
-		(net "/VOUT")
-	)
-	(via
 		(at 114.052031 113.59251)
 		(size 0.6)
@@
 	)
 	(via
-		(at 183.241631 116.456491)
-		(size 0.6)
-		(drill 0.3)
-		(layers "F.Cu" "B.Cu")
-		(free yes)
-		(net "/VOUT")
-	)
-	(via
 		(at 114.052031 115.163164)
 		(size 0.6)
@@
 	)
 	(via
-		(at 117.557231 115.213965)
-		(size 0.6)
-		(drill 0.3)
-		(layers "F.Cu" "B.Cu")
-		(free yes)
-		(net "/VOUT")
-	)
-	(via
 		(at 183.241631 118.027145)
 		(size 0.6)
@@
 	)
 	(via
-		(at 115.779231 118.355271)
-		(size 0.6)
-		(drill 0.3)
-		(layers "F.Cu" "B.Cu")
-		(free yes)
-		(net "/VOUT")
-	)
-	(via
-		(at 117.557231 118.355272)
-		(size 0.6)
-		(drill 0.3)
-		(layers "F.Cu" "B.Cu")
-		(free yes)
-		(net "/VOUT")
-	)
-	(via
-		(at 181.670977 129.054891)
-		(size 0.6)
-		(drill 0.3)
-		(layers "F.Cu" "B.Cu")
-		(free yes)
-		(net "/VOUT")
-	)
-	(via
 		(at 183.241631 114.885838)
 		(size 0.6)
@@
 	)
 	(via
-		(at 183.241631 119.597799)
-		(size 0.6)
-		(drill 0.3)
-		(layers "F.Cu" "B.Cu")
-		(free yes)
-		(net "/VOUT")
-	)
-	(via
-		(at 115.779231 115.213964)
-		(size 0.6)
-		(drill 0.3)
-		(layers "F.Cu" "B.Cu")
-		(free yes)
-		(net "/VOUT")
-	)
-	(via
 		(at 165.903145 118.336091)
 		(size 0.6)
@@
 	)
 	(via
-		(at 124.897598 67.840891)
-		(size 0.6)
-		(drill 0.3)
-		(layers "F.Cu" "B.Cu")
-		(free yes)
-		(net "/SOURCE")
-	)
-	(via
 		(at 129.502443 68.055288)
 		(size 0.6)
@@
 	)
 	(via
-		(at 127.995532 68.055288)
-		(size 0.6)
-		(drill 0.3)
-		(layers "F.Cu" "B.Cu")
-		(free yes)
-		(net "/SOURCE")
-	)
-	(via
 		(at 135.486479 68.025995)
 		(size 0.6)
@@
 	)
 	(via
-		(at 132.945898 66.621691)
-		(size 0.6)
-		(drill 0.3)
-		(layers "F.Cu" "B.Cu")
-		(free yes)
-		(net "/SOURCE")
-	)
-	(via
 		(at 135.255 70.621)
 		(size 0.8)
@@
 	)
 	(via
-		(at 129.96812 66.621691)
-		(size 0.6)
-		(drill 0.3)
-		(layers "F.Cu" "B.Cu")
-		(free yes)
-		(net "/SOURCE")
-	)
-	(via
 		(at 120.352721 66.286725)
 		(size 0.6)
@@
 	)
 	(via
-		(at 124.823121 66.286725)
-		(size 0.6)
-		(drill 0.3)
-		(layers "F.Cu" "B.Cu")
-		(free yes)
-		(net "/SOURCE")
-	)
-	(via
 		(at 136.271 70.621)
 		(size 0.8)
@@
 	)
 	(via
-		(at 131.009354 68.055288)
-		(size 0.6)
-		(drill 0.3)
-		(layers "F.Cu" "B.Cu")
-		(free yes)
-		(net "/SOURCE")
-	)
-	(via
 		(at 131.457009 66.621691)
 		(size 0.6)
@@
 	)
 	(via
-		(at 121.845343 66.286725)
-		(size 0.6)
-		(drill 0.3)
-		(layers "F.Cu" "B.Cu")
-		(free yes)
-		(net "/SOURCE")
-	)
-	(via
 		(at 132.516265 68.055288)
 		(size 0.6)
@@
 	)
 	(via
-		(at 121.883776 67.840891)
-		(size 0.6)
-		(drill 0.3)
-		(layers "F.Cu" "B.Cu")
-		(free yes)
-		(net "/SOURCE")
-	)
-	(via
 		(at 126.404509 67.840891)
 		(size 0.6)
@@
 		(polygon
 			(pts
-				(xy 129.608632 52.079) (xy 145.542 52.079) (xy 145.542 63.382) (xy 129.608632 63.382)
+				(xy 113.053632 52.079) (xy 145.542 52.079) (xy 145.542 63.195292) (xy 113.053632 63.195292)
 			)
 		)
@@
 		(polygon
 			(pts
-				(xy 119.995631 73.581291) (xy 119.995631 60.627291) (xy 126.858632 60.627291) (xy 126.858632 65.112383)
+				(xy 119.995631 73.581291) (xy 119.995631 64.605292) (xy 126.373632 64.605292) (xy 126.373632 64.583292)
 				(xy 127.869631 66.215291) (xy 133.838631 66.215291) (xy 137.013631 68.882291) (xy 137.013631 75.050292)
 				(xy 129.595 75.050292)
@@
 		(polygon
 			(pts
-				(xy 113.483632 113.150292) (xy 184.683632 113.150292) (xy 184.683632 121.659) (xy 113.483632 121.659)
+				(xy 113.483632 113.150292) (xy 184.683632 113.150292) (xy 184.683632 130.475292) (xy 113.483632 130.475292)
 			)
 		)
@@
 		(polygon
 			(pts
-				(xy 145.542 63.382) (xy 145.645 67.73) (xy 139.145 67.73) (xy 135.001 63.382)
+				(xy 145.535445 63.105292) (xy 145.644889 67.725292) (xy 139.995207 67.725292) (xy 132.127757 63.114492)
 			)
 		)
@@
 		(polygon
 			(pts
-				(xy 161.544 69.732) (xy 167.259 69.732) (xy 167.259 78.495) (xy 161.544 78.495)
+				(xy 161.544 69.732) (xy 175.583632 69.732) (xy 175.583632 78.495) (xy 161.544 78.495)
 			)
 		)
@@
 		(polygon
 			(pts
-				(xy 157.861 65.409) (xy 167.258632 65.409) (xy 167.258632 70.113) (xy 157.861 70.113)
+				(xy 157.861 65.409) (xy 175.583632 65.409) (xy 175.583632 70.113) (xy 157.861 70.113)
 			)
 		)
@@
 		(polygon
 			(pts
-				(xy 147.495 52.03) (xy 165.263 52.03) (xy 165.263 62.959) (xy 147.495 62.959)
+				(xy 147.495 52.03) (xy 182.953632 52.03) (xy 182.953632 62.959) (xy 147.495 62.959)
 			)
 		)
