File: Ai Sipder Bot Power System/LM5116 Kicad File/LM5116.kicad_sch (KiCad schematic)
At the start: 88 parts, among them J1 XT60-M, J10 PH1-01-UA, J11 PH1-01-UA, J12 PH1-01-UA, J13 PH1-01-UA, J14 61300311121, J15 61300311121, J16 61300311121, J17 61300311121, J18 61300311121, J19 61300311121, J2 PH1-01-UA, J20 61300311121, J21 61300311121, J22 61300311121, J23 61300311121, J24 61300311121, J25 61300311121, J3 PH1-01-UA, J4 PH1-01-UA, J5 PH1-01-UA, J6 PH1-01-UA, J7 PH1-01-UA, J8 PH1-01-UA, J9 PH1-01-UA, Q1 CSD17304Q3, Q2 CSD17304Q3, Q3 CSD17304Q3, Q4 CSD17304Q3, Q5 2N7002, Q6 IQDH29NE2LM5CG, U1 LM25116MHX/NOPB, U2 TLV1701AIDBVR, U3 TL431DBZ

Commit message: Expand the edgecut to satisfy 20H rule
Parts:
- C15: value 1u -> 2.2u
- C17: value 820n -> 2.2u
- C18: value 100n -> 2.2u
Changed lines of the file:
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@@
 			)
 		)
-		(property "Value" "820n"
+		(property "Value" "2.2u"
 			(at 264.16 90.1699 0)
 			(show_name no)
@@
 			)
 		)
-		(property "Value" "100n"
+		(property "Value" "2.2u"
 			(at 231.14 90.1699 0)
 			(show_name no)
@@
 			)
 		)
-		(property "Value" "1u"
+		(property "Value" "2.2u"
 			(at 241.3 90.1699 0)
 			(show_name no)

Commit message: Add schematic file
Parts:
- added J26: 691137710002, 691137710002:691137710002, symbol 691137710002:691137710002
- C15: value 2.2u -> 1u
- C17: value 2.2u -> 820n
- C18: value 2.2u -> 100n
Connections:
- net at F1.1, J1.P (POS): now also J26.2
- net at J1.N (NEG), Q6.5 (DRAIN1), Q6.6 (DRAIN2)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: now also J26.1
Changed lines of the file:
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@@
 	)
 	(junction
+		(at 308.61 201.295)
+		(diameter 0)
+		(color 0 0 0 0)
+	)
+	(junction
 		(at 213.36 203.2)
 		(diameter 0)
@@
 	)
 	(junction
+		(at 308.61 195.58)
+		(diameter 0)
+		(color 0 0 0 0)
+	)
+	(junction
 		(at 270.51 85.09)
 		(diameter 0)
@@
 	(wire
 		(pts
-			(xy 308.61 190.5) (xy 308.61 196.85)
+			(xy 308.61 190.5) (xy 308.61 195.58)
 		)
 		(stroke
@@
 	(wire
 		(pts
+			(xy 308.61 195.58) (xy 308.61 196.85)
+		)
+		(stroke
+			(width 0)
+			(type default)
+		)
+	)
+	(wire
+		(pts
 			(xy 64.77 100.965) (xy 64.77 102.87)
 		)
@@
 	(wire
 		(pts
+			(xy 308.61 201.295) (xy 308.61 219.71)
+		)
+		(stroke
+			(width 0)
+			(type default)
+		)
+	)
+	(wire
+		(pts
 			(xy 99.06 39.37) (xy 110.49 39.37)
 		)
@@
 	(wire
 		(pts
+			(xy 316.23 199.39) (xy 316.23 201.295)
+		)
+		(stroke
+			(width 0)
+			(type default)
+		)
+	)
+	(wire
+		(pts
 			(xy 182.88 163.83) (xy 182.88 172.72)
 		)
@@
 	(wire
 		(pts
+			(xy 316.23 195.58) (xy 308.61 195.58)
+		)
+		(stroke
+			(width 0)
+			(type default)
+		)
+	)
+	(wire
+		(pts
 			(xy 170.18 92.71) (xy 185.42 92.71)
 		)
@@
 	(wire
 		(pts
+			(xy 316.23 201.295) (xy 308.61 201.295)
+		)
+		(stroke
+			(width 0)
+			(type default)
+		)
+	)
+	(wire
+		(pts
 			(xy 281.94 97.79) (xy 281.94 104.14)
 		)
@@
 	(wire
 		(pts
-			(xy 308.61 219.71) (xy 308.61 199.39)
+			(xy 316.23 196.85) (xy 316.23 195.58)
+		)
+		(stroke
+			(width 0)
+			(type default)
+		)
+	)
+	(wire
+		(pts
+			(xy 308.61 199.39) (xy 308.61 201.295)
 		)
 		(stroke
@@
 			)
 		)
-		(property "Value" "2.2u"
+		(property "Value" "820n"
 			(at 264.16 90.1699 0)
 			(show_name no)
@@
 			)
 		)
-		(property "Value" "2.2u"
+		(property "Value" "100n"
 			(at 231.14 90.1699 0)
 			(show_name no)
@@
 			)
 		)
-		(property "Value" "2.2u"
+		(property "Value" "1u"
 			(at 241.3 90.1699 0)
 			(show_name no)
@@
 					(unit 1)
 				)
+			)
+		)
+	)
+	(symbol
+		(lib_id "691137710002:691137710002")
+		(at 321.31 196.85 270)
+		(mirror x)
+		(unit 1)
+		(body_style 1)
+		(exclude_from_sim no)
+		(in_bom yes)
+		(on_board yes)
+		(in_pos_files yes)
+		(dnp no)
+		(property "Reference" "J26"
+			(at 322.58 199.3901 90)
+			(show_name no)
+			(do_not_autoplace no)
+			(effects
+				(font
+					(size 1.27 1.27)
+				)
+				(justify left)
+			)
+		)
+		(property "Value" "691137710002"
+			(at 322.58 196.8501 90)
+			(show_name no)
+			(do_not_autoplace no)
+			(effects
+				(font
+					(size 1.27 1.27)
+				)
+				(justify left)
+			)
+		)
+		(property "Footprint" "691137710002:691137710002"
+			(at 321.31 196.85 0)
+			(hide yes)
+			(show_name no)
+			(do_not_autoplace no)
+			(effects
+				(font
+					(size 1.27 1.27)
+				)
+				(justify bottom)
+			)
+		)
+		(property "Datasheet" ""
+			(at 321.31 196.85 0)
+			(hide yes)
+			(show_name no)
+			(do_not_autoplace no)
+			(effects
+				(font
+					(size 1.27 1.27)
+				)
+			)
+		)
+		(property "Description" ""
+			(at 321.31 196.85 0)
+			(hide yes)
+			(show_name no)
+			(do_not_autoplace no)
+			(effects
+				(font
+					(size 1.27 1.27)
+				)
+			)
+		)
+		(pin "1"
+		)
+		(pin "2"
+		)
+		(instances
+			(project "LM5116"
+				(path "/31377078-18c6-42e8-84f6-8746c9c3df18"
+					(reference "J26")
+					(unit 1)
+				)

Commit message: Update Kicad File
Parts:
- Q1, Q2, Q3, Q4: footprint CSD17304Q3:DQG0008A -> NTTFS4C08NTAG:WDFN8_3P30X3P30_ONS
Changed lines of the file:
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@@
 			)
 		)
-		(property "Footprint" "CSD17304Q3:DQG0008A"
+		(property "Footprint" "NTTFS4C08NTAG:WDFN8_3P30X3P30_ONS"
 			(at 209.55 180.34 0)
 			(hide yes)
@@
 			)
 		)
-		(property "Footprint" "CSD17304Q3:DQG0008A"
+		(property "Footprint" "NTTFS4C08NTAG:WDFN8_3P30X3P30_ONS"
 			(at 88.9 194.31 0)
 			(hide yes)
@@
 			)
 		)
-		(property "Footprint" "CSD17304Q3:DQG0008A"
+		(property "Footprint" "NTTFS4C08NTAG:WDFN8_3P30X3P30_ONS"
 			(at 62.23 193.04 0)
 			(hide yes)
@@
 			)
 		)
-		(property "Footprint" "CSD17304Q3:DQG0008A"
+		(property "Footprint" "NTTFS4C08NTAG:WDFN8_3P30X3P30_ONS"
 			(at 179.07 180.34 0)
 			(hide yes)

Commit message: Update Kicad File
Connections:
- net GND: no longer C1.2, C10.2
- net GNDPWR: now also C1.2, C10.2
Changed lines of the file:
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@@
 	(symbol
 		(lib_id "power:GND")
-		(at 63.5 128.27 0)
-		(unit 1)
-		(body_style 1)
-		(exclude_from_sim no)
-		(in_bom yes)
-		(on_board yes)
-		(in_pos_files yes)
-		(dnp no)
-		(fields_autoplaced yes)
-		(property "Reference" "#PWR010"
-			(at 63.5 134.62 0)
-			(hide yes)
-			(show_name no)
-			(do_not_autoplace no)
-			(effects
-				(font
-					(size 1.27 1.27)
-				)
-			)
-		)
-		(property "Value" "GND"
-			(at 66.04 129.5399 0)
-			(show_name no)
-			(do_not_autoplace no)
-			(effects
-				(font
-					(size 1.27 1.27)
-				)
-				(justify left)
-			)
-		)
-		(property "Footprint" ""
-			(at 63.5 128.27 0)
-			(hide yes)
-			(show_name no)
-			(do_not_autoplace no)
-			(effects
-				(font
-					(size 1.27 1.27)
-				)
-			)
-		)
-		(property "Datasheet" ""
-			(at 63.5 128.27 0)
-			(hide yes)
-			(show_name no)
-			(do_not_autoplace no)
-			(effects
-				(font
-					(size 1.27 1.27)
-				)
-			)
-		)
-		(property "Description" "Power symbol creates a global label with name \"GND\" , ground"
-			(at 63.5 128.27 0)
-			(hide yes)
-			(show_name no)
-			(do_not_autoplace no)
-			(effects
-				(font
-					(size 1.27 1.27)
-				)
-			)
-		)
-		(pin "1"
-		)
-		(instances
-			(project "LM5116"
-				(path "/31377078-18c6-42e8-84f6-8746c9c3df18"
-					(reference "#PWR010")
-					(unit 1)
-				)
-			)
-		)
-	)
-	(symbol
-		(lib_id "power:GND")
 		(at 386.08 152.4 0)
 		(unit 1)
@@
 	(symbol
 		(lib_id "power:GNDPWR")
+		(at 214.63 52.07 0)
+		(unit 1)
+		(body_style 1)
+		(exclude_from_sim no)
+		(in_bom yes)
+		(on_board yes)
+		(in_pos_files yes)
+		(dnp no)
+		(fields_autoplaced yes)
+		(property "Reference" "#PWR022"
+			(at 214.63 57.15 0)
+			(hide yes)
+			(show_name no)
+			(do_not_autoplace no)
+			(effects
+				(font
+					(size 1.27 1.27)
+				)
+			)
+		)
+		(property "Value" "GNDPWR"
+			(at 214.503 55.88 0)
+			(show_name no)
+			(do_not_autoplace no)
+			(effects
+				(font
+					(size 1.27 1.27)
+				)
+			)
+		)
+		(property "Footprint" ""
+			(at 214.63 53.34 0)
+			(hide yes)
+			(show_name no)
+			(do_not_autoplace no)
+			(effects
+				(font
+					(size 1.27 1.27)
+				)
+			)
+		)
+		(property "Datasheet" ""
+			(at 214.63 53.34 0)
+			(hide yes)
+			(show_name no)
+			(do_not_autoplace no)
+			(effects
+				(font
+					(size 1.27 1.27)
+				)
+			)
+		)
+		(property "Description" "Power symbol creates a global label with name \"GNDPWR\" , global ground"
+			(at 214.63 52.07 0)
+			(hide yes)
+			(show_name no)
+			(do_not_autoplace no)
+			(effects
+				(font
+					(size 1.27 1.27)
+				)
+			)
+		)
+		(pin "1"
+		)
+		(instances
+			(project "LM5116"
+				(path "/31377078-18c6-42e8-84f6-8746c9c3df18"
+					(reference "#PWR022")
+					(unit 1)
+				)
+			)
+		)
+	)
+	(symbol
+		(lib_id "power:GNDPWR")
 		(at 213.36 223.52 0)
 		(unit 1)
@@
 	)
 	(symbol
-		(lib_id "power:GND")
-		(at 214.63 52.07 0)
-		(unit 1)
-		(body_style 1)
-		(exclude_from_sim no)
-		(in_bom yes)
-		(on_board yes)
-		(in_pos_files yes)
-		(dnp no)
-		(fields_autoplaced yes)
-		(property "Reference" "#PWR03"
-			(at 214.63 58.42 0)
-			(hide yes)
-			(show_name no)
-			(do_not_autoplace no)
-			(effects
-				(font
-					(size 1.27 1.27)
-				)
-			)
-		)
-		(property "Value" "GND"
-			(at 214.63 57.15 0)
-			(show_name no)
-			(do_not_autoplace no)
-			(effects
-				(font
-					(size 1.27 1.27)
-				)
-			)
-		)
-		(property "Footprint" ""
-			(at 214.63 52.07 0)
-			(hide yes)
-			(show_name no)
-			(do_not_autoplace no)
-			(effects
-				(font
-					(size 1.27 1.27)
-				)
-			)
-		)
-		(property "Datasheet" ""
-			(at 214.63 52.07 0)
-			(hide yes)
-			(show_name no)
-			(do_not_autoplace no)
-			(effects
-				(font
-					(size 1.27 1.27)
-				)
-			)
-		)
-		(property "Description" "Power symbol creates a global label with name \"GND\" , ground"
-			(at 214.63 52.07 0)
-			(hide yes)
-			(show_name no)
-			(do_not_autoplace no)
-			(effects
-				(font
-					(size 1.27 1.27)
-				)
-			)
-		)
-		(pin "1"
-		)
-		(instances
-			(project "LM5116"
-				(path "/31377078-18c6-42e8-84f6-8746c9c3df18"
-					(reference "#PWR03")
-					(unit 1)
-				)
-			)
-		)
-	)
-	(symbol
 		(lib_id "1 Pin Header:PH1-01-UA")
 		(at 361.95 38.1 270)
@@
 					(unit 1)
 				)
+			)
+		)
+	)
+	(symbol
+		(lib_id "power:GNDPWR")
+		(at 63.5 128.27 0)
+		(unit 1)
+		(body_style 1)
+		(exclude_from_sim no)
+		(in_bom yes)
+		(on_board yes)
+		(in_pos_files yes)
+		(dnp no)
+		(fields_autoplaced yes)
+		(property "Reference" "#PWR023"
+			(at 63.5 133.35 0)
+			(hide yes)
+			(show_name no)
+			(do_not_autoplace no)
+			(effects
+				(font
+					(size 1.27 1.27)
+				)
+			)
+		)
+		(property "Value" "GNDPWR"
+			(at 63.373 132.08 0)
+			(show_name no)
+			(do_not_autoplace no)
+			(effects
+				(font
+					(size 1.27 1.27)
+				)
+			)
+		)
+		(property "Footprint" ""
+			(at 63.5 129.54 0)
+			(hide yes)
+			(show_name no)
+			(do_not_autoplace no)
+			(effects
+				(font
+					(size 1.27 1.27)
+				)
+			)
+		)
+		(property "Datasheet" ""
+			(at 63.5 129.54 0)
+			(hide yes)
+			(show_name no)
+			(do_not_autoplace no)
+			(effects
+				(font
+					(size 1.27 1.27)
+				)
+			)
+		)
+		(property "Description" "Power symbol creates a global label with name \"GNDPWR\" , global ground"
+			(at 63.5 128.27 0)
+			(hide yes)
+			(show_name no)
+			(do_not_autoplace no)
+			(effects
+				(font
+					(size 1.27 1.27)
+				)
+			)
+		)
+		(pin "1"
+		)
+		(instances
+			(project "LM5116"
+				(path "/31377078-18c6-42e8-84f6-8746c9c3df18"
+					(reference "#PWR023")
+					(unit 1)
+				)

Commit message: Adjust VCC
Parts:
- C17: value 820n -> 2.2u
- C18: value 100n -> 2.2u
- R4: value 1Meg -> 0
Connections:
- net VOUT: no longer C1.1, U1.17 (VCCX)
- new net: C1.1, U1.17 (VCCX)
Changed lines of the file:
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@@
 	)
 	(junction
-		(at 214.63 36.83)
-		(diameter 0)
-		(color 0 0 0 0)
-	)
-	(junction
 		(at 74.93 114.3)
 		(diameter 0)
@@
 	(wire
 		(pts
-			(xy 214.63 36.83) (xy 224.79 36.83)
-		)
-		(stroke
-			(width 0)
-			(type default)
-		)
-	)
-	(wire
-		(pts
 			(xy 55.88 193.04) (xy 57.15 193.04)
 		)
@@
 		)
 	)
-	(label "VOUT"
-		(at 224.79 36.83 0)
-		(effects
-			(font
-				(size 1.27 1.27)
-			)
-			(justify left bottom)
-		)
-	)
 	(label "PGND"
 		(at 332.74 88.9 180)
@@
 			)
 		)
-		(property "Value" "820n"
+		(property "Value" "2.2u"
 			(at 264.16 90.1699 0)
 			(show_name no)
@@
 			)
 		)
-		(property "Value" "100n"
+		(property "Value" "2.2u"
 			(at 231.14 90.1699 0)
 			(show_name no)
@@
 			)
 		)
-		(property "Value" "1Meg"
+		(property "Value" "0"
 			(at 99.06 80.0099 0)
 			(show_name no)

Commit message: Update Kicad File
Parts:
- removed C1: 1u, Capacitor_SMD:C_0603_1608Metric_Pad1.08x0.95mm_HandSolder, symbol Device:C_US
- removed C12, C13: 150u, Capacitor_SMD:CP_Elec_10x10.5, symbol Device:C_Polarized_US
- removed J10, J11, J12, J13, J2, J3, J4, J5, J6, J7, J8, J9: PH1-01-UA, PH1_01_UA:CONN_PH1-01-UA_ADM, symbol 1 Pin Header:PH1-01-UA
- removed J14, J15, J16, J17, J18, J19, J20, J21, J22, J23, J24, J25: 61300311121, 61300311121:WURTH_61300311121, symbol 61300311121:61300311121
- removed J26: 691137710002, 691137710002:691137710002, symbol 691137710002:691137710002
- removed S1: 100SP1T1B4M2QE, SW_100SP1T1B4M2QE:SW_100SP1T1B4M2QE, symbol 100SP1T1B4M2QE:100SP1T1B4M2QE
- added C22, C23, C24: 2.2u, Capacitor_SMD:C_0603_1608Metric_Pad1.08x0.95mm_HandSolder, symbol Device:C
- added CR1: DFLT27A-7, DFLT27A_7:CR_LT27A-7_DIO, symbol DFLT27A-7:DFLT27A-7
- added CR2: SMBJ7.0CA-13-F, SMBJ7_0CA_13_F:SMB_DIO, symbol SMBJ7.0CA-13-F:SMBJ7.0CA-13-F
- added J1, J10, J11, J12, J2, J3, J4, J5, J6, J7, J8, J9: 61300411121, 61300411121:WURTH_61300411121, symbol 4 Pin Header:61300411121
- added J15: TB002V-500-02BE, TB002V-500-02B:CUI_TB002V-500-02BE, symbol TB002V-500-02BE:TB002V-500-02BE
- added SW1: EG1218, EG1218:SW_1218_EWI, symbol EG1218:EG1218
- C11, C14: value 150u -> 2200u; footprint Capacitor_SMD:CP_Elec_10x10.5 -> Capacitor_THT:CP_Radial_D10.0mm_P5.00mm
- C15: value 1u -> 2.2u
- C18, C2, C20: footprint Capacitor_SMD:C_0402_1005Metric_Pad0.74x0.62mm_HandSolder -> Capacitor_SMD:C_0603_1608Metric_Pad1.08x0.95mm_HandSolder
- C19, C21, C8: footprint Capacitor_SMD:C_0201_0603Metric_Pad0.64x0.40mm_HandSolder -> Capacitor_SMD:C_0603_1608Metric_Pad1.08x0.95mm_HandSolder
- C3: footprint Capacitor_SMD:C_0805_2012Metric_Pad1.18x1.45mm_HandSolder -> Capacitor_SMD:C_1206_3216Metric_Pad1.33x1.80mm_HandSolder
- C4: value 680u -> 1000u; footprint Capacitor_SMD:CP_Elec_10x10.5 -> Capacitor_THT:CP_Radial_D10.0mm_P5.00mm
- Q1, Q2, Q3, Q4: footprint NTTFS4C08NTAG:WDFN8_3P30X3P30_ONS -> CSD17304Q3:DQG0008A
- R11, R12, R13, R14, R15, R19, R21, R22, R23, R24, R25, R26, R27, R7: footprint Resistor_SMD:R_0402_1005Metric_Pad0.72x0.64mm_HandSolder -> Resistor_SMD:R_0603_1608Metric_Pad0.98x0.95mm_HandSolder
- R2, R20: footprint Resistor_SMD:R_0402_1005Metric_Pad0.72x0.64mm_HandSolder -> Resistor_SMD:R_0805_2012Metric_Pad1.20x1.40mm_HandSolder
- R3: footprint Resistor_SMD:R_0603_1608Metric_Pad0.98x0.95mm_HandSolder -> Resistor_SMD:R_0805_2012Metric_Pad1.20x1.40mm_HandSolder
- R4: value 0 -> 1Meg
- R6: value 140 -> 330
- renumbered J1 to J14
Connections:
- net EN: now also SW1.2
- net GND: now also C10.2
- net GNDPWR: now also U1.17 (VCCX), C22.2, C23.2, C24.2, CR1.2, CR2.2, J1.01, J10.01, J11.01, J12.01, J2.01, J3.01, J4.01, J5.01, J6.01, J7.01, J8.01, J9.01; no longer C10.2
- net SOURCE: now also C22.1, C23.1, C24.1, CR1.1
- net VOUT: now also CR2.1, J1.02, J10.02, J11.02, J12.02, J2.02, J3.02, J4.02, J5.02, J6.02, J7.02, J8.02, J9.02
- net at F1.1, J14.P (POS): now also J15.2
- net at R4.2: now also SW1.1
- net at J14.N (NEG), Q6.5 (DRAIN1), Q6.6 (DRAIN2)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: now also J15.1
- new net: J3.03, J3.04
- new net: J7.03, J7.04
- new net: J5.03, J5.04
- new net: J11.03, J11.04
- new net: J9.03, J9.04
- new net: J8.03, J8.04
- new net: J1.03, J1.04
- new net: J10.03, J10.04
- new net: J12.03, J12.04
- new net: J4.03, J4.04
- new net: J6.03, J6.04
- new net: J2.03, J2.04
Other:
- moved on the sheet: C21, Q3, Q4, R13, R14, R15, R17, R26, R27
