File: USB 2.0 HUB/USB 2.0 HUB/USB 2.0 HUB.kicad_pcb (KiCad board)
At the start: 4 copper layers, 66 x 52 mm, 58 parts, among them J1 USB-A-S-VT, J2 USB-A-S-VT, J3 USB4110GFA, U1 USB2512BT/M2, U3 AZ1117CH-3.3TRG1, U4 TPS2064DGNR, Y1 TSX-322524.0000MF15X-AC3

Commit message: Update Kicad File Footprint
Parts:
- added G***: LOGO, Hoshino:Reze, F.Cu at (125.1, 74.9)
- added G***: LOGO, BA:Cute, F.Cu at (159.1, 66.2)
- moved NT1 17.3 mm to (150.4, 62.8), turned to -45 degrees
Connections:
- U3 pad 4: GNDPWR -> /VDD33
Routing:
- net Net-(D3-A): track 127.1 -> 24.5 mm
- net /5V_FILTER: track 104.4 -> 27.9 mm
- net /VDDA33: track 95.6 -> 37.1 mm
- net Net-(D2-A): track 77.2 -> 42.7 mm
- net /VBUS: track 31.2 -> 21.0 mm
- net /VDD33: track 37.6 -> 42.9 mm
- net GNDPWR: track 33.5 -> 38.2 mm, vias 23 -> 21
- net GND: track 43.6 -> 45.3 mm
- added copper zone on In2.Cu, net /5V_FILTER
- added copper zone on In2.Cu, net /VBUS
- added copper zone on In2.Cu, net /VDDA33
- added copper zone on In2.Cu, net Net-(D2-A)
- added copper zone on In2.Cu, net Net-(D3-A)
Other:
- board text added: "USB 2.0 HUB VERSION 1.0"

Commit message: Update Kicad File And Result Image
Parts:
- removed R1: 634, Resistor_SMD:R_0603_1608Metric_Pad0.98x0.95mm_HandSolder
- removed R2: 1k, Resistor_SMD:R_0603_1608Metric_Pad0.98x0.95mm_HandSolder
- C10: value 2.2u -> 4.7u; footprint Capacitor_SMD:C_0603_1608Metric_Pad1.08x0.95mm_HandSolder -> Capacitor_SMD:C_0805_2012Metric_Pad1.18x1.45mm_HandSolder
- R8: value 330 -> 0
Connections:
- U3 pad 1: Net-(U3-ADJ/GND) -> GNDPWR
Routing:
- net Net-(U3-ADJ/GND): track 6.08 -> 0.00 mm
- net GNDPWR: track 38.2 -> 41.9 mm
- net /VDD33: track 42.9 -> 40.6 mm

Commit message: Update Kicad File
Connections:
- J3 pad A1/B12: CGND -> GND
- J3 pad A6: unconnected-(J3-DP1-PadA6) -> /DP1
- J3 pad A7: unconnected-(J3-DN1-PadA7) -> /DN1
- J3 pad B1/A12: CGND -> GND
Routing:
- net /VBUS: track 21.0 -> 15.5 mm, vias 2 -> 3
- net GND: track 45.3 -> 49.6 mm, vias 28 -> 30
- net CGND: track 32.7 -> 28.5 mm
- net /DN1: track 22.8 -> 25.1 mm
- net /DP1: track 22.9 -> 25.1 mm
Changed lines of the file:
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@@
 			(size 0.6 1.15)
 			(layers "F.Cu" "F.Mask" "F.Paste")
-			(net "CGND")
+			(net "GND")
 			(pinfunction "GND_A1/B12")
 			(pintype "power_in")
@@
 			(size 0.3 1.15)
 			(layers "F.Cu" "F.Mask" "F.Paste")
-			(net "unconnected-(J3-DP1-PadA6)")
+			(net "/DP1")
 			(pinfunction "DP1_A6")
-			(pintype "bidirectional+no_connect")
+			(pintype "bidirectional")
 			(solder_mask_margin 0.05)
 		)
@@
 			(size 0.3 1.15)
 			(layers "F.Cu" "F.Mask" "F.Paste")
-			(net "unconnected-(J3-DN1-PadA7)")
+			(net "/DN1")
 			(pinfunction "DN1_A7")
-			(pintype "bidirectional+no_connect")
+			(pintype "bidirectional")
 			(solder_mask_margin 0.05)
 		)
@@
 			(size 0.6 1.15)
 			(layers "F.Cu" "F.Mask" "F.Paste")
-			(net "CGND")
+			(net "GND")
 			(pinfunction "GND__1_B1/A12")
 			(pintype "power_in")
@@
 	)
 	(segment
+		(start 139.922091 41.14019)
+		(end 140.192742 40.869539)
+		(width 0.2113)
+		(layer "F.Cu")
+		(net "GND")
+	)
+	(segment
 		(start 150.020088 62.411967)
 		(end 150.011197 62.411967)
@@
 	)
 	(segment
+		(start 133.522091 41.14019)
+		(end 133.25144 40.869539)
+		(width 0.2113)
+		(layer "F.Cu")
+		(net "GND")
+	)
+	(segment
 		(start 124.535952 51.730865)
 		(end 125.375233 51.730865)
@@
 	)
 	(segment
+		(start 133.25144 39.754492)
+		(end 133.639768 39.366164)
+		(width 0.2113)
+		(layer "F.Cu")
+		(net "GND")
+	)
+	(segment
+		(start 139.687265 39.3192)
+		(end 139.5984 39.3192)
+		(width 0.2113)
+		(layer "F.Cu")
+		(net "GND")
+	)
+	(segment
+		(start 133.25144 40.869539)
+		(end 133.25144 39.754492)
+		(width 0.2113)
+		(layer "F.Cu")
+		(net "GND")
+	)
+	(segment
 		(start 143.065848 59.703048)
 		(end 143.2052 59.8424)
@@
 	)
 	(segment
+		(start 140.192742 40.869539)
+		(end 140.192742 39.824677)
+		(width 0.2113)
+		(layer "F.Cu")
+		(net "GND")
+	)
+	(segment
+		(start 140.192742 39.824677)
+		(end 139.687265 39.3192)
+		(width 0.2113)
+		(layer "F.Cu")
+		(net "GND")
+	)
+	(segment
 		(start 125.49272 52.687633)
 		(end 125.49272 53.4466)
@@
 	)
 	(via
+		(at 139.5984 39.3192)
+		(size 0.5)
+		(drill 0.3)
+		(layers "F.Cu" "B.Cu")
+		(net "GND")
+	)
+	(via
 		(at 127.508 43.942)
 		(size 0.6)
@@
 		(net "GND")
 	)
+	(via
+		(at 133.639768 39.366164)
+		(size 0.5)
+		(drill 0.3)
+		(layers "F.Cu" "B.Cu")
+		(net "GND")
+	)
 	(segment
 		(start 119.328702 52.673709)
@@
 	)
 	(segment
-		(start 138.927741 40.94584)
-		(end 139.122091 41.14019)
-		(width 0.2113)
-		(layer "F.Cu")
-		(net "/VBUS")
-	)
-	(segment
-		(start 134.516441 40.25954)
-		(end 138.927741 40.25954)
-		(width 0.2113)
-		(layer "F.Cu")
-		(net "/VBUS")
-	)
-	(segment
 		(start 139.171091 42.397091)
 		(end 139.954 43.18)
@@
 	)
 	(segment
-		(start 134.516441 40.94584)
-		(end 134.516441 40.25954)
+		(start 134.322091 41.14019)
+		(end 134.322091 41.953909)
+		(width 0.2113)
+		(layer "F.Cu")
+		(net "/VBUS")
+	)
+	(segment
+		(start 134.322091 41.953909)
+		(end 134.3152 41.9608)
 		(width 0.2113)
 		(layer "F.Cu")
@@
 		(net "/VBUS")
 	)
-	(segment
-		(start 134.322091 41.14019)
-		(end 134.516441 40.94584)
-		(width 0.2113)
-		(layer "F.Cu")
-		(net "/VBUS")
-	)
-	(segment
-		(start 138.927741 40.25954)
-		(end 138.927741 40.94584)
-		(width 0.2113)
-		(layer "F.Cu")
+	(via
+		(at 129.686246 46.086772)
+		(size 0.5)
+		(drill 0.3)
+		(layers "F.Cu" "B.Cu")
 		(net "/VBUS")
 	)
 	(via
-		(at 129.686246 46.086772)
+		(at 134.3152 41.9608)
 		(size 0.5)
 		(drill 0.3)
@@
 	)
 	(segment
+		(start 136.719972 40.367309)
+		(end 137.395309 40.367309)
+		(width 0.1)
+		(layer "F.Cu")
+		(net "/DN1")
+	)
+	(segment
 		(start 134.098454 48.431038)
 		(end 134.106919 48.422573)
@@
 	)
 	(segment
+		(start 137.472091 40.444091)
+		(end 137.472091 41.14019)
+		(width 0.1)
+		(layer "F.Cu")
+		(net "/DN1")
+	)
+	(segment
+		(start 136.472091 40.61519)
+		(end 136.719972 40.367309)
+		(width 0.1)
+		(layer "F.Cu")
+		(net "/DN1")
+	)
+	(segment
 		(start 135.343105 46.837165)
 		(end 135.343105 47.208106)
@@
 	)
 	(segment
+		(start 137.395309 40.367309)
+		(end 137.472091 40.444091)
+		(width 0.1)
+		(layer "F.Cu")
+		(net "/DN1")
+	)
+	(segment
 		(start 137.292091 44.212923)
 		(end 137.012091 44.212923)
@@
 	)
 	(segment
+		(start 136.472091 41.14019)
+		(end 136.472091 40.61519)
+		(width 0.1)
+		(layer "F.Cu")
+		(net "/DN1")
+	)
+	(segment
 		(start 136.772091 42.702691)
 		(end 136.772091 43.372923)
@@
 	)
 	(segment
+		(start 136.652 41.91)
+		(end 136.972091 41.589909)
+		(width 0.1)
+		(layer "F.Cu")
+		(net "/DP1")
+	)
+	(segment
 		(start 136.572091 42.602691)
 		(end 136.572091 46.053909)
@@
 	)
 	(segment
+		(start 135.972091 41.66519)
+		(end 136.216901 41.91)
+		(width 0.1)
+		(layer "F.Cu")
+		(net "/DP1")
+	)
+	(segment
 		(start 132.952199 58.55044)
 		(end 132.952199 58.762572)
@@
 	)
 	(segment
+		(start 136.216901 41.91)
+		(end 136.652 41.91)
+		(width 0.1)
+		(layer "F.Cu")
+		(net "/DP1")
+	)
+	(segment
 		(start 132.938229 46.522573)
 		(end 132.721694 46.522573)
@@
 	)
 	(segment
+		(start 136.972091 41.589909)
+		(end 136.972091 41.14019)
+		(width 0.1)
+		(layer "F.Cu")
+		(net "/DP1")
+	)
+	(segment
+		(start 135.972091 41.14019)
+		(end 135.972091 41.66519)
+		(width 0.1)
+		(layer "F.Cu")
+		(net "/DP1")
+	)
+	(segment
 		(start 132.507788 48.709208)
 		(end 132.507788 49.46879)
@@
 	)
 	(segment
-		(start 140.497091 40.56519)
-		(end 139.973091 41.08919)
-		(width 0.702)
-		(layer "F.Cu")
-		(net "CGND")
-	)
-	(segment
 		(start 141.530624 34.544)
 		(end 141.832091 34.845467)
@@
 	)
 	(segment
-		(start 133.471092 41.08919)
-		(end 133.471091 41.14019)
-		(width 0.702)
-		(layer "F.Cu")
-		(net "CGND")
-	)
-	(segment
 		(start 127.125213 38.794587)
 		(end 129.344636 38.794587)
@@
 	)
 	(segment
-		(start 141.832091 40.56519)
-		(end 140.497091 40.56519)
-		(width 0.702)
-		(layer "F.Cu")
-		(net "CGND")
-	)
-	(segment
 		(start 131.612091 35.265909)
 		(end 132.334 34.544)
@@
 	)
 	(segment
-		(start 139.973091 41.08919)
-		(end 139.973091 41.14019)
-		(width 0.702)
-		(layer "F.Cu")
-		(net "CGND")
-	)
-	(segment
 		(start 141.832091 34.845467)
 		(end 141.832091 36.63519)
@@
 	)
 	(segment
-		(start 131.612091 40.56519)
-		(end 132.947092 40.56519)
-		(width 0.702)
-		(layer "F.Cu")
-		(net "CGND")
-	)
-	(segment
 		(start 141.832091 36.63519)
 		(end 141.832091 40.56519)
@@
 		(width 0.702)
 		(layer "F.Cu")
-		(net "CGND")
-	)
-	(segment
-		(start 132.947092 40.56519)
-		(end 133.471092 41.08919)
-		(width 0.702)
-		(layer "F.Cu")
