File: USB 2.0 HUB/USB 2.0 HUB/USB 2.0 HUB.kicad_sch (KiCad schematic)
At the start: 58 parts, among them J1 USB-A-S-VT, J2 USB-A-S-VT, J3 USB4110GFA, U1 USB2512BT/M2, U3 AZ1117CH-3.3TRG1, U4 TPS2064DGNR, Y1 TSX-322524.0000MF15X-AC3

Commit message: Update Kicad File Footprint
Parts:
- removed R17: 0, Resistor_SMD:R_0402_1005Metric_Pad0.72x0.64mm_HandSolder, symbol Device:R_US
- added NT1: NetTie_2, NetTie:NetTie-2_SMD_Pad0.5mm, symbol Device:NetTie_2
- C10: value 2.2u -> 4.7u; footprint Capacitor_SMD:C_0603_1608Metric_Pad1.08x0.95mm_HandSolder -> Capacitor_SMD:C_0805_2012Metric_Pad1.18x1.45mm_HandSolder
Connections:
- net GND: now also NT1.1
- net GNDPWR: now also NT1.2; no longer U3.4 (EPAD)
- net VDD33: now also U3.4 (EPAD)
Changed lines of the file:
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@@
 	(wire
 		(pts
-			(xy 461.01 177.8) (xy 467.36 177.8)
+			(xy 461.01 177.8) (xy 468.63 177.8)
 		)
 		(stroke
@@
 	(wire
 		(pts
-			(xy 482.6 177.8) (xy 474.98 177.8)
+			(xy 482.6 177.8) (xy 473.71 177.8)
 		)
 		(stroke
@@
 	(wire
 		(pts
+			(xy 76.2 281.94) (xy 80.01 281.94)
+		)
+		(stroke
+			(width 0)
+			(type default)
+		)
+	)
+	(wire
+		(pts
 			(xy 441.325 327.66) (xy 441.325 313.69)
 		)
@@
 		)
 	)
+	(label "VDD33"
+		(at 76.2 281.94 180)
+		(effects
+			(font
+				(size 1.27 1.27)
+			)
+			(justify right bottom)
+		)
+	)
 	(label "XTALOUT"
 		(at 299.72 201.93 0)
@@
 	)
 	(symbol
-		(lib_id "Device:R_US")
-		(at 471.17 177.8 90)
-		(unit 1)
-		(body_style 1)
-		(exclude_from_sim no)
-		(in_bom yes)
-		(on_board yes)
-		(in_pos_files yes)
-		(dnp no)
-		(fields_autoplaced yes)
-		(property "Reference" "R17"
-			(at 471.17 171.45 90)
-			(show_name no)
-			(do_not_autoplace no)
-			(effects
-				(font
-					(size 1.27 1.27)
-				)
-			)
-		)
-		(property "Value" "0"
-			(at 471.17 173.99 90)
-			(show_name no)
-			(do_not_autoplace no)
-			(effects
-				(font
-					(size 1.27 1.27)
-				)
-			)
-		)
-		(property "Footprint" "Resistor_SMD:R_0402_1005Metric_Pad0.72x0.64mm_HandSolder"
-			(at 471.424 176.784 90)
-			(hide yes)
-			(show_name no)
-			(do_not_autoplace no)
-			(effects
-				(font
-					(size 1.27 1.27)
-				)
-			)
-		)
-		(property "Datasheet" ""
-			(at 471.17 177.8 0)
-			(hide yes)
-			(show_name no)
-			(do_not_autoplace no)
-			(effects
-				(font
-					(size 1.27 1.27)
-				)
-			)
-		)
-		(property "Description" "Resistor, US symbol"
-			(at 471.17 177.8 0)
-			(hide yes)
-			(show_name no)
-			(do_not_autoplace no)
-			(effects
-				(font
-					(size 1.27 1.27)
-				)
-			)
-		)
-		(pin "1"
-		)
-		(pin "2"
-		)
-		(instances
-			(project "USB 2.0 HUB"
-				(path "/a1b0b12d-4135-4cc2-b5a1-d3c289e0357e"
-					(reference "R17")
-					(unit 1)
-				)
-			)
-		)
-	)
-	(symbol
 		(lib_id "TSX-322524.0000MF15X-AC3:TSX-322524.0000MF15X-AC3")
 		(at 510.54 234.95 0)
@@
 	)
 	(symbol
+		(lib_id "Device:NetTie_2")
+		(at 471.17 177.8 0)
+		(unit 1)
+		(body_style 1)
+		(exclude_from_sim no)
+		(in_bom no)
+		(on_board yes)
+		(in_pos_files yes)
+		(dnp no)
+		(fields_autoplaced yes)
+		(property "Reference" "NT1"
+			(at 471.17 172.72 0)
+			(show_name no)
+			(do_not_autoplace no)
+			(effects
+				(font
+					(size 1.27 1.27)
+				)
+			)
+		)
+		(property "Value" "NetTie_2"
+			(at 471.17 175.26 0)
+			(show_name no)
+			(do_not_autoplace no)
+			(effects
+				(font
+					(size 1.27 1.27)
+				)
+			)
+		)
+		(property "Footprint" "NetTie:NetTie-2_SMD_Pad0.5mm"
+			(at 471.17 177.8 0)
+			(hide yes)
+			(show_name no)
+			(do_not_autoplace no)
+			(effects
+				(font
+					(size 1.27 1.27)
+				)
+			)
+		)
+		(property "Datasheet" ""
+			(at 471.17 177.8 0)
+			(hide yes)
+			(show_name no)
+			(do_not_autoplace no)
+			(effects
+				(font
+					(size 1.27 1.27)
+				)
+			)
+		)
+		(property "Description" "Net tie, 2 pins"
+			(at 471.17 177.8 0)
+			(hide yes)
+			(show_name no)
+			(do_not_autoplace no)
+			(effects
+				(font
+					(size 1.27 1.27)
+				)
+			)
+		)
+		(pin "2"
+		)
+		(pin "1"
+		)
+		(instances
+			(project "USB 2.0 HUB"
+				(path "/a1b0b12d-4135-4cc2-b5a1-d3c289e0357e"
+					(reference "NT1")
+					(unit 1)
+				)
+			)
+		)
+	)
+	(symbol
 		(lib_id "power:GND")
 		(at 500.38 232.41 270)
@@
 	)
 	(symbol
-		(lib_id "power:GNDPWR")
-		(at 80.01 281.94 0)
-		(unit 1)
-		(body_style 1)
-		(exclude_from_sim no)
-		(in_bom yes)
-		(on_board yes)
-		(in_pos_files yes)
-		(dnp no)
-		(fields_autoplaced yes)
-		(property "Reference" "#PWR059"
-			(at 80.01 287.02 0)
-			(hide yes)
-			(show_name no)
-			(do_not_autoplace no)
-			(effects
-				(font
-					(size 1.27 1.27)
-				)
-			)
-		)
-		(property "Value" "GNDPWR"
-			(at 79.883 285.75 0)
-			(show_name no)
-			(do_not_autoplace no)
-			(effects
-				(font
-					(size 1.27 1.27)
-				)
-			)
-		)
-		(property "Footprint" ""
-			(at 80.01 283.21 0)
-			(hide yes)
-			(show_name no)
-			(do_not_autoplace no)
-			(effects
-				(font
-					(size 1.27 1.27)
-				)
-			)
-		)
-		(property "Datasheet" ""
-			(at 80.01 283.21 0)
-			(hide yes)
-			(show_name no)
-			(do_not_autoplace no)
-			(effects
-				(font
-					(size 1.27 1.27)
-				)
-			)
-		)
-		(property "Description" "Power symbol creates a global label with name \"GNDPWR\" , global ground"
-			(at 80.01 281.94 0)
-			(hide yes)
-			(show_name no)
-			(do_not_autoplace no)
-			(effects
-				(font
-					(size 1.27 1.27)
-				)
-			)
-		)
-		(pin "1"
-		)
-		(instances
-			(project "USB 2.0 HUB"
-				(path "/a1b0b12d-4135-4cc2-b5a1-d3c289e0357e"
-					(reference "#PWR059")
-					(unit 1)
-				)
-			)
-		)
-	)
-	(symbol
 		(lib_id "power:GND")
 		(at 104.14 154.94 0)
@@
 			)
 		)
-		(property "Value" "2.2u"
+		(property "Value" "4.7u"
 			(at 179.07 286.0039 0)
 			(show_name no)
@@
 			)
 		)
-		(property "Footprint" "Capacitor_SMD:C_0603_1608Metric_Pad1.08x0.95mm_HandSolder"
+		(property "Footprint" "Capacitor_SMD:C_0805_2012Metric_Pad1.18x1.45mm_HandSolder"
 			(at 175.26 284.48 0)
 			(hide yes)

Commit message: Update Kicad File And Result Image
Parts:
- removed R1: 634, Resistor_SMD:R_0603_1608Metric_Pad0.98x0.95mm_HandSolder, symbol Device:R_US
- removed R2: 1k, Resistor_SMD:R_0603_1608Metric_Pad0.98x0.95mm_HandSolder, symbol Device:R_US
- R8: value 330 -> 0
Connections:
- net GNDPWR: now also U3.1 (ADJ/GND)
Changed lines of the file:
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@@
 	)
 	(junction
-		(at 139.7 279.4)
-		(diameter 0)
-		(color 0 0 0 0)
-	)
-	(junction
 		(at 31.75 279.4)
 		(diameter 0)
@@
 	)
 	(junction
-		(at 139.7 294.64)
-		(diameter 0)
-		(color 0 0 0 0)
-	)
-	(junction
 		(at 165.1 279.4)
 		(diameter 0)
@@
 	(wire
 		(pts
-			(xy 139.7 292.1) (xy 139.7 294.64)
-		)
-		(stroke
-			(width 0)
-			(type default)
-		)
-	)
-	(wire
-		(pts
 			(xy 91.44 151.13) (xy 93.98 151.13)
 		)
@@
 	(wire
 		(pts
-			(xy 133.985 294.64) (xy 139.7 294.64)
+			(xy 133.985 294.64) (xy 137.16 294.64)
 		)
 		(stroke
@@
 	(wire
 		(pts
-			(xy 139.7 279.4) (xy 152.4 279.4)
-		)
-		(stroke
-			(width 0)
-			(type default)
-		)
-	)
-	(wire
-		(pts
 			(xy 410.21 201.295) (xy 410.21 203.2)
 		)
@@
 	(wire
 		(pts
-			(xy 130.81 279.4) (xy 139.7 279.4)
+			(xy 130.81 279.4) (xy 152.4 279.4)
 		)
 		(stroke
@@
 	(wire
 		(pts
-			(xy 139.7 294.64) (xy 139.7 297.18)
-		)
-		(stroke
-			(width 0)
-			(type default)
-		)
-	)
-	(wire
-		(pts
 			(xy 530.86 220.98) (xy 530.86 232.41)
 		)
@@
 	(wire
 		(pts
-			(xy 139.7 304.8) (xy 139.7 307.34)
-		)
-		(stroke
-			(width 0)
-			(type default)
-		)
-	)
-	(wire
-		(pts
 			(xy 119.38 132.08) (xy 121.92 132.08)
 		)
@@
 	(wire
 		(pts
-			(xy 139.7 279.4) (xy 139.7 284.48)
-		)
-		(stroke
-			(width 0)
-			(type default)
-		)
-	)
-	(wire
-		(pts
 			(xy 439.42 325.12) (xy 445.77 325.12)
 		)
@@
 	(symbol
 		(lib_id "power:GNDPWR")
-		(at 139.7 307.34 0)
+		(at 137.16 294.64 0)
 		(unit 1)
 		(body_style 1)
@@
 		(fields_autoplaced yes)
 		(property "Reference" "#PWR050"
-			(at 139.7 312.42 0)
+			(at 137.16 299.72 0)
 			(hide yes)
 			(show_name no)
@@
 		)
 		(property "Value" "GNDPWR"
-			(at 139.573 311.15 0)
+			(at 137.033 298.45 0)
 			(show_name no)
 			(do_not_autoplace no)
@@
 		)
 		(property "Footprint" ""
-			(at 139.7 308.61 0)
+			(at 137.16 295.91 0)
 			(hide yes)
 			(show_name no)
@@
 		)
 		(property "Datasheet" ""
-			(at 139.7 308.61 0)
+			(at 137.16 295.91 0)
 			(hide yes)
 			(show_name no)
@@
 		)
 		(property "Description" "Power symbol creates a global label with name \"GNDPWR\" , global ground"
-			(at 139.7 307.34 0)
+			(at 137.16 294.64 0)
 			(hide yes)
 			(show_name no)
@@
 			)
 		)
-		(property "Value" "330"
+		(property "Value" "0"
 			(at 97.79 142.24 90)
 			(show_name no)
@@
 	)
 	(symbol
-		(lib_id "Device:R_US")
-		(at 139.7 288.29 0)
-		(unit 1)
-		(body_style 1)
-		(exclude_from_sim no)
-		(in_bom yes)
-		(on_board yes)
-		(in_pos_files yes)
-		(dnp no)
-		(fields_autoplaced yes)
-		(property "Reference" "R1"
-			(at 142.24 287.0199 0)
-			(show_name no)
-			(do_not_autoplace no)
-			(effects
-				(font
-					(size 1.27 1.27)
-				)
-				(justify left)
-			)
-		)
-		(property "Value" "634"
-			(at 142.24 289.5599 0)
-			(show_name no)
-			(do_not_autoplace no)
-			(effects
-				(font
-					(size 1.27 1.27)
-				)
-				(justify left)
-			)
-		)
-		(property "Footprint" "Resistor_SMD:R_0603_1608Metric_Pad0.98x0.95mm_HandSolder"
-			(at 140.716 288.544 90)
-			(hide yes)
-			(show_name no)
-			(do_not_autoplace no)
-			(effects
-				(font
-					(size 1.27 1.27)
-				)
-			)
-		)
-		(property "Datasheet" ""
-			(at 139.7 288.29 0)
-			(hide yes)
-			(show_name no)
-			(do_not_autoplace no)
-			(effects
-				(font
-					(size 1.27 1.27)
-				)
-			)
-		)
-		(property "Description" "Resistor, US symbol"
-			(at 139.7 288.29 0)
-			(hide yes)
-			(show_name no)
-			(do_not_autoplace no)
-			(effects
-				(font
-					(size 1.27 1.27)
-				)
-			)
-		)
-		(pin "2"
-		)
-		(pin "1"
-		)
-		(instances
-			(project "USB 2.0 HUB"
-				(path "/a1b0b12d-4135-4cc2-b5a1-d3c289e0357e"
-					(reference "R1")
-					(unit 1)
-				)
-			)
-		)
-	)
-	(symbol
 		(lib_id "power:GND")
 		(at 520.7 237.49 0)
@@
 					(unit 1)
 				)
-			)
-		)
-	)
-	(symbol
-		(lib_id "Device:R_US")
-		(at 139.7 300.99 0)
-		(unit 1)
-		(body_style 1)
-		(exclude_from_sim no)
-		(in_bom yes)
-		(on_board yes)
-		(in_pos_files yes)
-		(dnp no)
-		(fields_autoplaced yes)
-		(property "Reference" "R2"
-			(at 142.24 299.7199 0)
-			(show_name no)
-			(do_not_autoplace no)
-			(effects
-				(font
-					(size 1.27 1.27)
-				)
-				(justify left)
-			)
-		)
-		(property "Value" "1k"
-			(at 142.24 302.2599 0)
-			(show_name no)
-			(do_not_autoplace no)
-			(effects
-				(font
-					(size 1.27 1.27)
-				)
-				(justify left)
-			)
-		)
-		(property "Footprint" "Resistor_SMD:R_0603_1608Metric_Pad0.98x0.95mm_HandSolder"
-			(at 140.716 301.244 90)
-			(hide yes)
-			(show_name no)
-			(do_not_autoplace no)
-			(effects
-				(font
-					(size 1.27 1.27)
-				)
-			)
-		)
-		(property "Datasheet" ""
-			(at 139.7 300.99 0)
-			(hide yes)
-			(show_name no)
-			(do_not_autoplace no)
-			(effects
-				(font
-					(size 1.27 1.27)
-				)
-			)
-		)
-		(property "Description" "Resistor, US symbol"
-			(at 139.7 300.99 0)
-			(hide yes)
-			(show_name no)
-			(do_not_autoplace no)
-			(effects
-				(font
-					(size 1.27 1.27)
-				)
-			)
-		)
-		(pin "1"
-		)
-		(pin "2"
-		)
-		(instances
-			(project "USB 2.0 HUB"
-				(path "/a1b0b12d-4135-4cc2-b5a1-d3c289e0357e"
-					(reference "R2")
-					(unit 1)
-				)

Commit message: Update Kicad File
Parts:
- R8: value 0 -> 330
Connections:
- net CGND: no longer J3.A1/B12 (GND), J3.B1/A12 (GND__1)
- net DN1: now also J3.A7 (DN1)
- net DP1: now also J3.A6 (DP1)
- net GND: now also J3.A1/B12 (GND), J3.B1/A12 (GND__1)
- no-connect marks 10 -> 8
Changed lines of the file:
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@@
 	)
 	(junction
+		(at 104.14 146.05)
+		(diameter 0)
+		(color 0 0 0 0)
+	)
+	(junction
 		(at 379.73 295.91)
 		(diameter 0)
@@
 	)
 	(junction
-		(at 91.44 135.89)
-		(diameter 0)
-		(color 0 0 0 0)
-	)
-	(junction
 		(at 153.67 113.03)
 		(diameter 0)
@@
 	)
 	(junction
-		(at 91.44 138.43)
+		(at 410.21 201.295)
 		(diameter 0)
 		(color 0 0 0 0)
 	)
 	(junction
-		(at 410.21 201.295)
+		(at 91.44 135.89)
 		(diameter 0)
 		(color 0 0 0 0)
@@
 	)
 	(no_connect
-		(at 53.34 123.19)
-	)
-	(no_connect
 		(at 474.98 279.4)
 	)
@@
 	)
 	(no_connect
-		(at 53.34 120.65)
-	)
-	(no_connect
 		(at 88.9 128.27)
 	)
@@
 	(wire
 		(pts
-			(xy 91.44 135.89) (xy 91.44 138.43)
+			(xy 94.615 115.57) (xy 94.615 113.03)
 		)
 		(stroke
@@
 	(wire
 		(pts
-			(xy 94.615 115.57) (xy 94.615 113.03)
+			(xy 121.92 124.46) (xy 121.92 129.54)
 		)
 		(stroke
@@
 	(wire
 		(pts
-			(xy 121.92 124.46) (xy 121.92 129.54)
+			(xy 488.95 237.49) (xy 497.84 237.49)
 		)
 		(stroke
@@
 	(wire
 		(pts
-			(xy 488.95 237.49) (xy 497.84 237.49)
+			(xy 149.86 212.09) (xy 151.13 212.09)
 		)
 		(stroke
@@
 	(wire
 		(pts
-			(xy 149.86 212.09) (xy 151.13 212.09)
+			(xy 104.14 135.89) (xy 104.14 146.05)
 		)
 		(stroke
@@
 	(wire
 		(pts
-			(xy 91.44 133.35) (xy 91.44 135.89)
-		)
-		(stroke
-			(width 0)
-			(type default)
-		)
-	)
-	(wire
-		(pts
 			(xy 389.89 288.29) (xy 389.89 284.48)
 		)
@@
 	(wire
 		(pts
+			(xy 91.44 135.89) (xy 104.14 135.89)
+		)
+		(stroke
+			(width 0)
+			(type default)
+		)
+	)
+	(wire
+		(pts
 			(xy 477.52 281.94) (xy 477.52 290.83)
 		)
@@
 	(wire
 		(pts
+			(xy 91.44 133.35) (xy 91.44 135.89)
+		)
+		(stroke
+			(width 0)
+			(type default)
+		)
+	)
+	(wire
+		(pts
 			(xy 486.41 325.12) (xy 486.41 311.15)
 		)
@@
 		)
 	)
+	(label "DP1"
+		(at 53.34 120.65 180)
+		(effects
+			(font
+				(size 1.27 1.27)
+			)
+			(justify right bottom)
+		)
+	)
 	(label "VDD33"
 		(at 172.72 224.79 180)
@@
 		)
 	)
+	(label "DN1"
+		(at 53.34 123.19 180)
+		(effects
+			(font
+				(size 1.27 1.27)
+			)
+			(justify right bottom)
+		)
+	)
 	(label "OCS_N2"
 		(at 355.6 316.23 0)
@@
 			)
 		)
-		(property "Value" "0"
+		(property "Value" "330"
 			(at 97.79 142.24 90)
 			(show_name no)
